Commit message: added pulsed terrain mapping

File: pomo_description/urdf/simple.urdf.xacro (robot description, xacro)
@@ -126,4 +126,77 @@
 		<child link="right_camera_optical"/>
 	</joint>
+	<link name="lidar_link">
+		<inertial>
+			<origin xyz="0 0 0" rpy="0 0 0"/>
+			<mass value="${cm}" />
+			<xacro:box_inertia x="${cs}" y="${cs}" z="${cs}" mass="${cm}"/>
+		</inertial>
+		<visual>
+			<origin xyz="0 0 0" rpy="0 0 0"/>
+			<geometry>
+				<box size="${cs} ${cs} ${cs}"/>
+			</geometry>
+		</visual>
+		<collision>
+			<origin xyz="0 0 0" rpy="0 0 0"/>
+			<geometry>
+				<box size="${cs} ${cs} ${cs}"/>
+			</geometry>
+		</collision>
+	</link>
+	<joint name="lidar_joint" type="revolute"> <!-- configurable angle -->
+		<limit upper="${pi/2}" lower="${-pi/2}" velocity="${0.1*pi}" effort="10000000"/>
+		<pose>0 0 0 0 0 0</pose>
+		<origin
+			xyz="${0.55*lx} 0 ${-0.3*lz}"
+			rpy="0 0 0" />
+		<parent
+			link="base_link" />
+		<child
+			link="lidar_link" />
+		<axis
+			xyz="0 1 0" rpy="0 0 0"/>
+	</joint>
+	<transmission name="lidar_transmission">
+		<type>transmission_interface/SimpleTransmission</type>
+		<actuator name="lidar_servo">
+			<hardwareInterface>hardware_interface/EffortJointInterface</hardwareInterface>
+			<mechanicalReduction>1</mechanicalReduction>
+		</actuator>
+		<joint name="lidar_joint">
+			<hardwareInterface>hardware_interface/EffortJointInterface</hardwareInterface>
+		</joint>
+	</transmission>
+	<gazebo reference="lidar_link">
+		<sensor type="ray" name="lidar">
+			<pose>0 0 0 0 0 0</pose>
+			<visualize>true</visualize> <!-- ?? -->
+			<update_rate>40</update_rate>
+			<ray>
+				<scan>
+					<horizontal>
+						<samples>1024</samples>
+						<resolution>1</resolution><!--?-->
+						<min_angle>-2.35</min_angle> <!-- +-135 deg -->
+						<max_angle>2.35</max_angle>
+					</horizontal>
+				</scan>
+				<range>
+					<min>0.06</min>
+					<max>4.0</max>
+					<resolution>0.01</resolution>
+				</range>
+				<noise>
+					<type>gaussian</type>
+					<mean>0.0</mean>
+					<stddev>0.01</stddev>
+				</noise>
+			</ray>
+			<plugin name="gazebo_ros_head_hokuyo_controller" filename="libgazebo_ros_laser.so">
+				<topicName>scan</topicName>
+				<frameName>lidar_link</frameName>
+			</plugin>
+		</sensor>
+	</gazebo>
 	<xacro:wheel wheel_prefix="left" wheel_mass="${wm}" wheel_radius="${wr}" wheel_thickness="${wt}" parent="base_link">
 		<origin xyz="0 ${0.5*wd} ${-0.5*lz}" rpy="0 0 0"/>

Commit message: simpler urdf

File: pomo_description/urdf/simple.urdf.xacro (robot description, xacro)
@@ -12,6 +12,7 @@
 	<xacro:property name="cs" value="0.01"/> <!-- camera size ... -->
 	<xacro:property name="cm" value="0.1"/> <!-- camera mass ... -->
-	<xacro:property name="ch" value="0.0"/> <!-- camera height, deg -->
-	<xacro:property name="ca" value="20.0"/> <!-- camera pitch, deg -->
+	<xacro:property name="ch" value="${20*inch}"/> <!-- camera height (from ground) -->
+	<xacro:property name="ca" value="45.0"/> <!-- camera pitch, deg -->
+	<xacro:property name="cd" value="${12*inch}"/> <!-- stereo camera distance (baseline), m -->
 	<xacro:property name="wd" value="${24*inch}"/> <!-- wheel separation -->
 	<xacro:property name="wr" value="${0.5*14.3*inch}"/> <!-- wheel radius -->
@@ -71,5 +72,5 @@
 		type="fixed">
 		<origin
-			xyz="${0.5*lx} ${0.5*ly} ${0.5*lz}"
+			xyz="${0.5*lx} ${0.5*cd} ${ch-0.5*lz-wr}"
 			rpy="0 ${ca*deg} 0" />
 		<parent
@@ -110,5 +111,5 @@
 		type="fixed">
 		<origin
-			xyz="${0.5*lx} ${-0.5*ly} ${0.5*lz}"
+			xyz="${0.5*lx} ${-0.5*cd} ${ch-0.5*lz-wr}"
 			rpy="0 ${ca*deg} 0" />
 		<parent
@@ -285,6 +286,82 @@
 				<cameraInfoTopicName>camera_info</cameraInfoTopicName>
 				<frameName>right_camera_optical</frameName>
+				<hackBaseline>${cd}</hackBaseline>
 			</plugin>
 		</sensor>
 	</gazebo>
+	<link name="kinect_link">
+		<inertial>
+			<origin xyz="0 0 0" rpy="0 0 0"/>
+			<mass value="${cm}" />
+			<xacro:box_inertia x="${cs}" y="${cs}" z="${cs}" mass="${cm}"/>
+		</inertial>
+		<visual>
+			<origin xyz="0 0 0" rpy="0 0 0"/>
+			<geometry>
+				<box size="${cs} ${cs} ${cs}"/>
+			</geometry>
+		</visual>
+		<collision>
+			<origin xyz="0 0 0" rpy="0 0 0"/>
+			<geometry>
+				<box size="${cs} ${cs} ${cs}"/>
+			</geometry>
+		</collision>
+	</link>
+	<joint
+		name="kinect_joint"
+		type="fixed">
+		<origin
+			xyz="${0.5*lx} 0 ${0.5*lz}"
+			rpy="0 ${ca*deg} 0" />
+		<parent
+			link="base_link" />
+		<child
+			link="kinect_link" />
+		<axis
+			xyz="0 1 0" />
+	</joint>
+	<link name="kinect_optical">
+	</link>
+	<joint name="kinect_optical_joint" type="fixed">
+		<origin xyz="0 0 0" rpy="${-pi/2} 0 ${-pi/2}"/>
+		<parent link="kinect_link"/>
+		<child link="kinect_optical"/>
+	</joint>
+    <gazebo reference="kinect_link">
+      <sensor type="depth" name="kinect">
+        <always_on>true</always_on>
+        <update_rate>20.0</update_rate>
+        <camera>
+          <horizontal_fov>${60.0*deg}</horizontal_fov>
+          <image>
+            <format>B8G8R8</format>
+            <width>640</width>
+            <height>480</height>
+          </image>
+          <clip>
+            <near>0.05</near>
+            <far>8.0</far>
+          </clip>
+        </camera>
+        <plugin name="kinect_camera_controller" filename="libgazebo_ros_openni_kinect.so">
+          <cameraName>kinect</cameraName>
+          <alwaysOn>true</alwaysOn>
+          <updateRate>10</updateRate>
+          <imageTopicName>rgb/image_raw</imageTopicName>
+          <depthImageTopicName>depth/image_raw</depthImageTopicName>
+          <pointCloudTopicName>depth/points</pointCloudTopicName>
+          <cameraInfoTopicName>rgb/camera_info</cameraInfoTopicName>
+          <depthImageCameraInfoTopicName>depth/camera_info</depthImageCameraInfoTopicName>
+          <frameName>kinect_optical</frameName>
+          <baseline>0.1</baseline>
+          <distortion_k1>0.0</distortion_k1>
+          <distortion_k2>0.0</distortion_k2>
+          <distortion_k3>0.0</distortion_k3>
+          <distortion_t1>0.0</distortion_t1>
+          <distortion_t2>0.0</distortion_t2>
+          <pointCloudCutoff>0.4</pointCloudCutoff>
+        </plugin>
+      </sensor>
+    </gazebo>
 </robot>

Commit message: todo: add noisy depth camera plugin

File: pomo_description/urdf/simple.urdf.xacro (robot description, xacro)
@@ -81,11 +81,11 @@
 			xyz="0 1 0" />
 	</joint>
-	  <joint name="left_camera_optical_joint" type="fixed">
+	<joint name="left_camera_optical_joint" type="fixed">
 		<origin xyz="0 0 0" rpy="${-pi/2} 0 ${-pi/2}"/>
 		<parent link="left_camera"/>
 		<child link="left_camera_optical"/>
-	  </joint>
-	  <link name="left_camera_optical">
-	  </link>
+	</joint>
+	<link name="left_camera_optical">
+	</link>
 	<link name="right_camera">
 		<inertial>
@@ -329,39 +329,45 @@
 		<child link="kinect_optical"/>
 	</joint>
-    <gazebo reference="kinect_link">
-      <sensor type="depth" name="kinect">
-        <always_on>true</always_on>
-        <update_rate>20.0</update_rate>
-        <camera>
-          <horizontal_fov>${60.0*deg}</horizontal_fov>
-          <image>
-            <format>B8G8R8</format>
-            <width>640</width>
-            <height>480</height>
-          </image>
-          <clip>
-            <near>0.05</near>
-            <far>8.0</far>
-          </clip>
-        </camera>
-        <plugin name="kinect_camera_controller" filename="libgazebo_ros_openni_kinect.so">
-          <cameraName>kinect</cameraName>
-          <alwaysOn>true</alwaysOn>
-          <updateRate>10</updateRate>
-          <imageTopicName>rgb/image_raw</imageTopicName>
-          <depthImageTopicName>depth/image_raw</depthImageTopicName>
-          <pointCloudTopicName>depth/points</pointCloudTopicName>
-          <cameraInfoTopicName>rgb/camera_info</cameraInfoTopicName>
-          <depthImageCameraInfoTopicName>depth/camera_info</depthImageCameraInfoTopicName>
-          <frameName>kinect_optical</frameName>
-          <baseline>0.1</baseline>
-          <distortion_k1>0.0</distortion_k1>
-          <distortion_k2>0.0</distortion_k2>
-          <distortion_k3>0.0</distortion_k3>
-          <distortion_t1>0.0</distortion_t1>
-          <distortion_t2>0.0</distortion_t2>
-          <pointCloudCutoff>0.4</pointCloudCutoff>
-        </plugin>
-      </sensor>
-    </gazebo>
+	<gazebo reference="kinect_link">
+		<sensor type="depth" name="kinect">
+			<always_on>true</always_on>
+			<update_rate>20.0</update_rate>
+			<camera>
+				<horizontal_fov>${60.0*deg}</horizontal_fov>
+				<image>
+					<format>B8G8R8</format>
+					<width>640</width>
+					<height>480</height>
+				</image>
+				<clip>
+					<near>0.05</near>
+					<far>8.0</far>
+				</clip>
+				<!-- WARNING : no noise in depth -->
+				<noise>
+					<type>gaussian</type>
+					<mean>0.0</mean>
+					<stddev>0.01</stddev>
+				</noise>
+			</camera>
+			<plugin name="kinect_camera_controller" filename="libgazebo_ros_openni_kinect.so">
+				<cameraName>kinect</cameraName>
+				<alwaysOn>true</alwaysOn>
+				<updateRate>10</updateRate>
+				<imageTopicName>rgb/image_raw</imageTopicName>
+				<depthImageTopicName>depth/image_raw</depthImageTopicName>
+				<pointCloudTopicName>depth/points</pointCloudTopicName>
+				<cameraInfoTopicName>rgb/camera_info</cameraInfoTopicName>
+				<depthImageCameraInfoTopicName>depth/camera_info</depthImageCameraInfoTopicName>
+				<frameName>kinect_optical</frameName>
+				<baseline>0.1</baseline>
+				<distortion_k1>0.0</distortion_k1>
+				<distortion_k2>0.0</distortion_k2>
+				<distortion_k3>0.0</distortion_k3>
+				<distortion_t1>0.0</distortion_t1>
+				<distortion_t2>0.0</distortion_t2>
+				<pointCloudCutoff>0.4</pointCloudCutoff>
+			</plugin>
+		</sensor>
+	</gazebo>
 </robot>
