Commit message: update URDF + add working IMU code

File: pwm_description/urdf/WheelchairDev.SLDASM.urdf (robot description, URDF)
Before this commit: robot wheelchair, 15 links, 14 joints
Links:
- removed link base_footprint
- removed link realsense_optical
- link back_link: mass 21.3849460447243 -> 22.009; geometry collision mesh filename=package://WheelchairDev.SLDASM/meshes/back_link.STL; visual mesh filename=package://WheelchairDev.SLDASM/meshes/back_link.STL
- link base_link: mass 98.4139630936699 -> 98.414; geometry collision mesh filename=package://WheelchairDev.SLDASM/meshes/base_link.STL; visual mesh filename=package://WheelchairDev.SLDASM/meshes/base_link.STL
- link caster_bl_link: mass ${2.0*lb} -> 1.2339; geometry collision mesh filename=package://WheelchairDev.SLDASM/meshes/caster_bl_link.STL; visual mesh filename=package://WheelchairDev.SLDASM/meshes/caster_bl_link.STL
- link caster_br_link: mass ${2.0*lb} -> 98.414; geometry collision mesh filename=package://WheelchairDev.SLDASM/meshes/caster_br_link.STL; visual mesh filename=package://WheelchairDev.SLDASM/meshes/caster_br_link.STL
- link caster_fl_link: mass ${2.0*lb} -> 1.2339; geometry collision mesh filename=package://WheelchairDev.SLDASM/meshes/caster_fl_link.STL; visual mesh filename=package://WheelchairDev.SLDASM/meshes/caster_fl_link.STL
- link caster_fr_link: mass ${2.0*lb} -> 1.2339; geometry collision mesh filename=package://WheelchairDev.SLDASM/meshes/caster_fr_link.STL; visual mesh filename=package://WheelchairDev.SLDASM/meshes/caster_fr_link.STL
- link footrest_link: mass 2.24583004981917 -> 2.3451; geometry collision mesh filename=package://WheelchairDev.SLDASM/meshes/footrest_link.STL; visual mesh filename=package://WheelchairDev.SLDASM/meshes/footrest_link.STL
- link gps_link: mass 0.026768 -> 0.032213; geometry collision mesh filename=package://WheelchairDev.SLDASM/meshes/gps_link.STL; visual mesh filename=package://WheelchairDev.SLDASM/meshes/gps_link.STL
- link left_wheel_link: mass ${4.0*lb} -> 3.7492; geometry collision mesh filename=package://WheelchairDev.SLDASM/meshes/left_wheel_link.STL; visual mesh filename=package://WheelchairDev.SLDASM/meshes/left_wheel_link.STL
- link lidar_link: geometry collision mesh filename=package://WheelchairDev.SLDASM/meshes/lidar_link.STL; visual mesh filename=package://WheelchairDev.SLDASM/meshes/lidar_link.STL
- link realsense_link: geometry collision mesh filename=package://WheelchairDev.SLDASM/meshes/realsense_link.STL; visual mesh filename=package://WheelchairDev.SLDASM/meshes/realsense_link.STL
- link right_wheel_link: mass ${4.0*lb} -> 3.7492; geometry collision mesh filename=package://WheelchairDev.SLDASM/meshes/right_wheel_link.STL; visual mesh filename=package://WheelchairDev.SLDASM/meshes/right_wheel_link.STL
- link seat_link: mass 39.8904807609114 -> 39.89; geometry collision mesh filename=package://WheelchairDev.SLDASM/meshes/seat_link.STL; visual mesh filename=package://WheelchairDev.SLDASM/meshes/seat_link.STL
Joints:
- removed joint base_footprint_joint
- removed joint realsense_optical_joint
- joint back_joint: limit (none) -> effort=0 velocity=0; origin xyz=-0.23495 0 0.127 rpy=1.5707963267949 0 0 -> xyz=-0.23495 0 0.127 rpy=1.5708 0 0; type fixed -> revolute
- joint caster_bl_joint: type fixed -> continuous
- joint caster_br_joint: type fixed -> continuous
- joint caster_fl_joint: type fixed -> continuous
- joint caster_fr_joint: type fixed -> continuous
- joint footrest_joint: limit (none) -> effort=0 velocity=0; origin xyz=0.2667 0 0.0317500000000001 rpy=1.5707963267949 0 0 -> xyz=0.2667 0 0.03175 rpy=1.5708 0 0; type fixed -> revolute
- joint gps_joint: axis 0 0 1 -> 0 0 0
- joint lidar_joint: axis 0 0 1 -> 0 0 0; origin xyz=0.13695 -0.32488 -0.00060405 rpy=-1.5708 8.2132E-18 0.026657 -> xyz=0.13695 -0.32488 -0.00060405 rpy=-1.5708 -4.1826E-18 0.026657
- joint realsense_joint: axis 0 0 1 -> 0 0 0
- joint seat_joint: limit lower=0.0 upper=0.3 effort=1500 velocity=0.5 -> effort=0 velocity=0; origin xyz=0.0889000000000003 -0.0126999999999997 0.50361 rpy=0 0 0 -> xyz=0.0889 -0.0127 0.50361 rpy=0 0 0
