Commit message: reasonable urdf configuration

File: pwm_description/urdf/defs.urdf.xacro (robot description, xacro)
@@ -18,3 +18,8 @@
 			izz="${0.0833333 * mass * (x*x + y*y)}" />
 	</xacro:macro>
+    <xacro:macro name="sphere_inertia" params="r m">
+		<inertia ixx="${0.4*m*r*r}" ixy="0.0" ixz="0.0"
+			iyy="${0.4*m*r*r}" iyz="0.0"
+			izz="${0.4*m*r*r}" />
+    </xacro:macro>
 </robot>

File: pwm_description/urdf/wheelchairdev.urdf.xacro (robot description, xacro)
@@ -1,6 +1,15 @@
 <?xml version="1.0"?>
 <robot name="wheelchair" xmlns:xacro="http://ros.org/wiki/xacro">
+    <xacro:arg name="sim" default="false"/>
     <xacro:include filename="$(find pwm_description)/urdf/defs.urdf.xacro"/>
     <xacro:include filename="$(find pwm_description)/urdf/wheelchairdev.gazebo"/>
+    <xacro:macro name="alias" params="src dst">
+        <link name="${dst}" />
+        <joint name="alias_${src}_${dst}" type="fixed">
+            <origin xyz="0 0 0" rpy="0 0 0"/>
+            <parent link="${src}"/>
+            <child link="${dst}"/>
+        </joint>
+    </xacro:macro>
     <link name="base_footprint">
     </link>
@@ -16,7 +25,6 @@
                 xyz="-5.97916491205108E-05 -5.55111512312578E-17 0.153027812315766"
                 rpy="0 0 0" />
-            <mass
-                value="98.4139630936699" />
-            <xacro:box_inertia x="1e-3" y="1e-3" z="1e-3" mass="1e-3"/>
+            <mass value="98.4139630936699" />
+            <xacro:box_inertia x="0.711" y="0.457" z="0.305" mass="98.4"/>
         </inertial>
         <visual>
@@ -141,5 +149,5 @@
     <joint
         name="footrest_joint"
-        type="fixed">
+        type="fixed"> <!-- TODO : technically revolute, broken for our chair -->
         <origin
             xyz="0.2667 0 0.0317500000000001"
@@ -256,30 +264,15 @@
         <child link="camera_optical"/>
     </joint>
-    <!-- alignment frames -->
     <!-- setup aliases for compatibility with realsense -->
-    <link name="camera_aligned_depth_to_color_frame"/>
-    <joint name="align_d2c" type="fixed">
-        <origin xyz="0 0 0" rpy="0 0 0"/>
-        <parent link="camera_optical"/>
-        <child link="camera_aligned_depth_to_color_frame"/>
-    </joint>
-    <link name="camera_aligned_depth_to_infra1_frame"/>
-    <joint name="align_d2i1" type="fixed">
-        <origin xyz="0 0 0" rpy="0 0 0"/>
-        <parent link="camera_optical"/>
-        <child link="camera_aligned_depth_to_infra1_frame"/>
-    </joint>
-    <link name="camera_aligned_depth_to_infra2_frame"/>
-    <joint name="align_d2i2" type="fixed">
-        <origin xyz="0 0 0" rpy="0 0 0"/>
-        <parent link="camera_optical"/>
-        <child link="camera_aligned_depth_to_infra2_frame"/>
-    </joint>
-    <link name="camera_aligned_depth_to_fisheye_frame" />
-    <joint name="align_d2f" type="fixed">
-        <origin xyz="0 0 0" rpy="0 0 0"/>
-        <parent link="camera_optical"/>
-        <child link="camera_aligned_depth_to_fisheye_frame"/>
-    </joint>
+    <xacro:if value="$(arg sim)">
+        <xacro:alias src="camera_link" dst="camera_color_frame"/>
+        <xacro:alias src="camera_link" dst="camera_depth_frame"/>
+        <xacro:alias src="camera_link" dst="camera_infra1_frame"/>
+        <xacro:alias src="camera_link" dst="camera_infra2_frame"/>
+        <xacro:alias src="camera_optical" dst="camera_color_optical_frame"/>
+        <xacro:alias src="camera_optical" dst="camera_depth_optical_frame"/>
+        <xacro:alias src="camera_optical" dst="camera_infra2_optical_frame"/>
+        <xacro:alias src="camera_optical" dst="camera_infra1_optical_frame"/>
+    </xacro:if>
     <link
         name="back_link">
@@ -321,5 +314,5 @@
     <joint
         name="back_joint"
-        type="fixed">
+        type="revolute">
         <origin
             xyz="-0.23495 0 0.127"
@@ -331,7 +324,5 @@
         <axis
             xyz="0 0 -1" />
-        <!--
         <limit lower="-3.14" upper="3.14" effort="1500" velocity="0.5" />
-        -->
     </joint>
     <link
@@ -485,5 +476,5 @@
             <mass
                 value="${2.0*lb}" />
-            <xacro:cylinder_inertia m="${2.0*lb}" r="${0.5*8*inch}" h="${2.0*inch}"/>
+            <xacro:sphere_inertia m="${2.0*lb}" r="${0.5*8*inch}"/>
         </inertial>
         <visual>
@@ -511,6 +502,11 @@
             </geometry>
             -->
+            <!--
             <geometry>
                 <cylinder length="${2.0*inch}" radius="${0.5*8*inch}"/>
+            </geometry>
+            -->
+            <geometry>
+                <sphere radius="${0.5*8*inch}"/>
             </geometry>
         </collision>
@@ -537,5 +533,5 @@
             <mass
                 value="${2.0*lb}" />
-            <xacro:cylinder_inertia m="${2.0*lb}" r="${0.5*8*inch}" h="${2.0*inch}"/>
+            <xacro:sphere_inertia m="${2.0*lb}" r="${0.5*8*inch}"/>
         </inertial>
         <visual>
@@ -557,6 +553,11 @@
                 xyz="0 0 0"
                 rpy="0 0 0" />
+            <!--
             <geometry>
                 <cylinder length="${2.0*inch}" radius="${0.5*8*inch}"/>
+            </geometry>
+            -->
+            <geometry>
+                <sphere radius="${0.5*8*inch}"/>
             </geometry>
         </collision>
@@ -583,5 +584,5 @@
             <mass
                 value="${2.0*lb}" />
-            <xacro:cylinder_inertia m="${2.0*lb}" r="${0.5*8*inch}" h="${2.0*inch}"/>
+            <xacro:sphere_inertia m="${2.0*lb}" r="${0.5*8*inch}"/>
         </inertial>
         <visual>
@@ -603,6 +604,11 @@
                 xyz="0 0 0"
                 rpy="0 0 0" />
+            <!--
             <geometry>
                 <cylinder length="${2.0*inch}" radius="${0.5*8*inch}"/>
+            </geometry>
+            -->
+            <geometry>
+                <sphere radius="${0.5*8*inch}"/>
             </geometry>
         </collision>
@@ -629,5 +635,5 @@
             <mass
                 value="${2.0*lb}" />
-            <xacro:cylinder_inertia m="${2.0*lb}" r="${0.5*8*inch}" h="${2.0*inch}"/>
+            <xacro:sphere_inertia m="${2.0*lb}" r="${0.5*8*inch}"/>
         </inertial>
         <visual>
@@ -649,6 +655,11 @@
                 xyz="0 0 0"
                 rpy="0 0 0" />
+            <!--
             <geometry>
                 <cylinder length="${2.0*inch}" radius="${0.5*8*inch}"/>
+            </geometry>
+            -->
+            <geometry>
+                <sphere radius="${0.5*8*inch}"/>
             </geometry>
         </collision>
@@ -668,4 +679,26 @@
     </joint>
     <!-- transmission -->
+    <transmission name="right_wheel_transmission">
+        <type>transmission_interface/SimpleTransmission</type>
+        <!--<type>hardware_interface</type>-->
+        <actuator name="right_wheel_motor">
+            <hardwareInterface>hardware_interface/VelocityJointInterface</hardwareInterface>
+            <mechanicalReduction>1</mechanicalReduction>
+        </actuator>
+        <joint name="right_wheel_joint">
+            <hardwareInterface>hardware_interface/VelocityJointInterface</hardwareInterface>
+        </joint>
+    </transmission>
+    <transmission name="left_wheel_transmission">
+        <type>transmission_interface/SimpleTransmission</type>
+        <!--<type>hardware_interface</type>-->
+        <actuator name="left_wheel_motor">
+            <hardwareInterface>hardware_interface/VelocityJointInterface</hardwareInterface>
+            <mechanicalReduction>1</mechanicalReduction>
+        </actuator>
+        <joint name="left_wheel_joint">
+            <hardwareInterface>hardware_interface/VelocityJointInterface</hardwareInterface>
+        </joint>
+    </transmission>
     <transmission name="seat_transmission">
         <type>transmission_interface/SimpleTransmission</type>
@@ -678,3 +711,13 @@
         </joint>
     </transmission>
+    <transmission name="back_transmission">
+        <type>transmission_interface/SimpleTransmission</type>
+        <actuator name="back_motor">
+            <hardwareInterface>hardware_interface/VelocityJointInterface</hardwareInterface>
+            <mechanicalReduction>1</mechanicalReduction>
+        </actuator>
+        <joint name="back_joint">
+            <hardwareInterface>hardware_interface/VelocityJointInterface</hardwareInterface>
+        </joint>
+    </transmission>
 </robot>
