Commit message: preliminary setup

File: pwm_description/urdf/wheelchairdev.urdf.xacro (robot description, xacro)
@@ -1,683 +1,781 @@
 <?xml version="1.0"?>
-<robot
-  name="wheelchair">
-  <link
-    name="base_link">
-    <inertial>
-      <origin
-        xyz="-5.97916491205108E-05 -5.55111512312578E-17 0.153027812315766"
-        rpy="0 0 0" />
-      <mass
-        value="98.4139630936699" />
-      <inertia
-        ixx="0"
-        ixy="0"
-        ixz="0"
-        iyy="0"
-        iyz="0"
-        izz="0" />
-    </inertial>
-    <visual>
-      <origin
-        xyz="0 0 0"
-        rpy="0 0 0" />
-      <geometry>
-        <mesh
-          filename="package://pwm_description/meshes/base_link.STL" />
-      </geometry>
-      <material
-        name="">
-        <color
-          rgba="0.792156862745098 0.819607843137255 0.933333333333333 1" />
-      </material>
-    </visual>
-    <collision>
-      <origin
-        xyz="0 0 0"
-        rpy="0 0 0" />
-      <geometry>
-        <mesh
-          filename="package://pwm_description/meshes/base_link.STL" />
-      </geometry>
-    </collision>
-  </link>
-  <link
-    name="seat_link">
-    <inertial>
-      <origin
-        xyz="-0.0332097722373201 0.00406938602338047 0.0228912507671721"
-        rpy="0 0 0" />
-      <mass
-        value="39.8904807609114" />
-      <inertia
-        ixx="0.122921824576847"
-        ixy="0.0164619739758286"
-        ixz="-0.146470483923146"
-        iyy="0.316753450399423"
-        iyz="0.0119623440768997"
-        izz="0.196633649371876" />
-    </inertial>
-    <visual>
-      <origin
-        xyz="0 0 0"
-        rpy="0 0 0" />
-      <geometry>
-        <mesh
-          filename="package://pwm_description/meshes/seat_link.STL" />
-      </geometry>
-      <material
-        name="">
-        <color
-          rgba="0.792156862745098 0.819607843137255 0.933333333333333 1" />
-      </material>
-    </visual>
-    <collision>
-      <origin
-        xyz="0 0 0"
-        rpy="0 0 0" />
-      <geometry>
-        <mesh
-          filename="package://pwm_description/meshes/seat_link.STL" />
-      </geometry>
-    </collision>
-  </link>
-  <joint
-    name="seat_joint"
-    type="prismatic">
-    <origin
-      xyz="0.0889000000000003 -0.0126999999999997 0.486604140008077"
-      rpy="0 0 0" />
-    <parent
-      link="base_link" />
-    <child
-      link="seat_link" />
-    <axis
-      xyz="0 0 1" />
-  <limit lower="0.0" upper="0.3" effort="1500" velocity="0.5" />
-  </joint>
-  <link
-    name="footrest_link">
-    <inertial>
-      <origin
-        xyz="0.0529952413391824 -0.208791421878138 -2.07915156937022E-05"
-        rpy="0 0 0" />
-      <mass
-        value="2.24583004981917" />
-      <inertia
-        ixx="0.00172839866541921"
-        ixy="0.000772961959349029"
-        ixz="3.16929282986145E-06"
-        iyy="0.00047716278384899"
-        iyz="-6.88732971243823E-06"
-        izz="0.00207972567905554" />
-    </inertial>
-    <visual>
-      <origin
-        xyz="0 0 0"
-        rpy="0 0 0" />
-      <geometry>
-        <mesh
-          filename="package://pwm_description/meshes/footrest_link.STL" />
-      </geometry>
-      <material
-        name="">
-        <color
-          rgba="0.792156862745098 0.819607843137255 0.933333333333333 1" />
-      </material>
-    </visual>
-    <collision>
-      <origin
-        xyz="0 0 0"
-        rpy="0 0 0" />
-      <geometry>
-        <mesh
-          filename="package://pwm_description/meshes/footrest_link.STL" />
-      </geometry>
-    </collision>
-  </link>
-  <joint
-    name="footrest_joint"
-    type="revolute">
-    <origin
-      xyz="0.2667 0 0.0317500000000001"
-      rpy="1.5707963267949 0 0" />
-    <parent
-      link="seat_link" />
-    <child
-      link="footrest_link" />
-    <axis
-      xyz="0 0 -1" />
-    <limit lower="-3.14" upper="3.14" effort="1500" velocity="0.5" />
-  </joint>
-  <link
-    name="lidar_link">
-    <inertial>
-      <origin
-        xyz="-0.0028645 3.9558E-06 -0.019418"
-        rpy="0 0 0" />
-      <mass
-        value="0.13624" />
-      <inertia
-        ixx="4.024E-05"
-        ixy="1.4318E-08"
-        ixz="-6.2254E-08"
-        iyy="4.1714E-05"
-        iyz="1.0354E-08"
-        izz="1.4743E-06" />
-    </inertial>
-    <visual>
-      <origin
-        xyz="0 0 0"
-        rpy="0 0 0" />
-      <geometry>
-        <mesh
-          filename="package://pwm_description/meshes/lidar_link.STL" />
-      </geometry>
-      <material
-        name="">
-        <color
-          rgba="0.79216 0.81961 0.93333 1" />
-      </material>
-    </visual>
-    <collision>
-      <origin
-        xyz="0 0 0"
-        rpy="0 0 0" />
-      <geometry>
-        <mesh
-          filename="package://pwm_description/meshes/lidar_link.STL" />
-      </geometry>
-    </collision>
-  </link>
-  <joint
-    name="lidar_joint"
-    type="fixed">
-    <origin
-      xyz="0.12479 -0.32059 -0.0006325"
-      rpy="-1.5708 8.2132E-18 0.24657" />
-    <parent
-      link="footrest_link" />
-    <child
-      link="lidar_link" />
-    <axis
-      xyz="0 0 0" />
-  </joint>
-  <link
-    name="realsense_link">
-    <inertial>
-      <origin
-        xyz="-0.012211 0.001403 8.0403E-05"
-        rpy="0 0 0" />
-      <mass
-        value="0.050576" />
-      <inertia
-        ixx="0"
-        ixy="0"
-        ixz="0"
-        iyy="0"
-        iyz="0"
-        izz="0" />
-    </inertial>
-    <visual>
-      <origin
-        xyz="0 0 0"
-        rpy="0 0 0" />
-      <geometry>
-        <mesh
-          filename="package://pwm_description/meshes/realsense_link.STL" />
-      </geometry>
-      <material
-        name="">
-        <color
-          rgba="0.66667 0.69804 0.76863 1" />
-      </material>
-    </visual>
-    <collision>
-      <origin
-        xyz="0 0 0"
-        rpy="0 0 0" />
-      <geometry>
-        <mesh
-          filename="package://pwm_description/meshes/realsense_link.STL" />
-      </geometry>
-    </collision>
-  </link>
-  <joint
-    name="realsense_joint"
-    type="fixed">
-    <origin
-      xyz="0.085027 -0.19321 0.00127"
-      rpy="-1.5708 3.2649E-15 0.24657" />
-    <parent
-      link="footrest_link" />
-    <child
-      link="realsense_link" />
-    <axis
-      xyz="0 0 0" />
-  </joint>
-  <link
-    name="back_link">
-    <inertial>
-      <origin
-        xyz="0.0595257246778351 0.272632134746619 0.0154465067130335"
-        rpy="0 0 0" />
-      <mass
-        value="21.3849460447243" />
-      <inertia
-        ixx="0.638823322523092"
-        ixy="-0.0353788477032128"
-        ixz="-0.147324675628681"
-        iyy="0.612040467785112"
-        iyz="0.00497982785800062"
-        izz="0.731113551637578" />
-    </inertial>
-    <visual>
-      <origin
-        xyz="0 0 0"
-        rpy="0 0 0" />
-      <geometry>
-        <mesh
-          filename="package://pwm_description/meshes/back_link.STL" />
-      </geometry>
-      <material
-        name="">
-        <color
-          rgba="0.792156862745098 0.819607843137255 0.933333333333333 1" />
-      </material>
-    </visual>
-    <collision>
-      <origin
-        xyz="0 0 0"
-        rpy="0 0 0" />
-      <geometry>
-        <mesh
-          filename="package://pwm_description/meshes/back_link.STL" />
-      </geometry>
-    </collision>
-  </link>
-  <joint
-    name="back_joint"
-    type="revolute">
-    <origin
-      xyz="-0.23495 0 0.127"
-      rpy="1.5707963267949 0 0" />
-    <parent
-      link="seat_link" />
-    <child
-      link="back_link" />
-    <axis
-      xyz="0 0 -1" />
-    <limit lower="-3.14" upper="3.14" effort="1500" velocity="0.5" />
-  </joint>
-  <link
-    name="gps_link">
-    <inertial>
-      <origin
-        xyz="-0.00076953 4.8962E-08 -0.010538"
-        rpy="0 0 0" />
-      <mass
-        value="0.026768" />
-      <inertia
-        ixx="0"
-        ixy="0"
-        ixz="0"
-        iyy="0"
-        iyz="0"
-        izz="0" />
-    </inertial>
-    <visual>
-      <origin
-        xyz="0 0 0"
-        rpy="0 0 0" />
-      <geometry>
-        <mesh
-          filename="package://pwm_description/meshes/gps_link.STL" />
-      </geometry>
-      <material
-        name="">
-        <color
-          rgba="0.29804 0.29804 0.29804 1" />
-      </material>
-    </visual>
-    <collision>
-      <origin
-        xyz="0 0 0"
-        rpy="0 0 0" />
-      <geometry>
-        <mesh
-          filename="package://pwm_description/meshes/gps_link.STL" />
-      </geometry>
-    </collision>
-  </link>
-  <joint
-    name="gps_joint"
-    type="fixed">
-    <origin
-      xyz="-0.050953 0.64 0.00030078"
-      rpy="-1.5708 -1.7107E-16 0.10298" />
-    <parent
-      link="back_link" />
-    <child
-      link="gps_link" />
-    <axis
-      xyz="0 0 0" />
-  </joint>
-  <link
-    name="right_wheel_link">
-    <inertial>
-      <origin
-        xyz="4.9960036108132E-16 -5.96744875736022E-16 0.0322019895391621"
-        rpy="0 0 0" />
-      <mass
-        value="3.25468436767915" />
-      <inertia
-        ixx="0"
-        ixy="0"
-        ixz="0"
-        iyy="0"
-        iyz="0"
-        izz="0" />
-    </inertial>
-    <visual>
-      <origin
-        xyz="0 0 0"
-        rpy="0 0 0" />
-      <geometry>
-        <mesh
-          filename="package://pwm_description/meshes/right_wheel_link.STL" />
-      </geometry>
-      <material
-        name="">
-        <color
-          rgba="0.792156862745098 0.819607843137255 0.933333333333333 1" />
-      </material>
-    </visual>
-    <collision>
-      <origin
-        xyz="0 0 0"
-        rpy="0 0 0" />
-      <geometry>
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
Commit message: functional sim

File: pwm_description/urdf/wheelchairdev.urdf.xacro (robot description, xacro)
@@ -139,5 +139,5 @@
     <joint
         name="footrest_joint"
-        type="revolute">
+        type="fixed">
         <origin
             xyz="0.2667 0 0.0317500000000001"
@@ -149,5 +149,7 @@
         <axis
             xyz="0 0 -1" />
+        <!--
         <limit lower="-3.14" upper="3.14" effort="1500" velocity="0.5" />
+        -->
     </joint>
     <link
@@ -202,5 +204,5 @@
             link="lidar_link" />
         <axis
-            xyz="0 0 0" />
+            xyz="0 0 1" />
     </joint>
     <link
@@ -249,6 +251,13 @@
             link="realsense_link" />
         <axis
-            xyz="0 0 0" />
-    </joint>
+            xyz="0 0 1" />
+    </joint>
+    <!-- optical frame -->
+    <link name="realsense_optical"/>
+	<joint name="realsense_optical_joint" type="fixed">
+		<origin xyz="0 0 0" rpy="${-pi/2} 0 ${-pi/2}"/>
+		<parent link="realsense_link"/>
+		<child link="realsense_optical"/>
+	</joint>
     <link
         name="back_link">
@@ -293,5 +302,5 @@
     <joint
         name="back_joint"
-        type="revolute">
+        type="fixed">
         <origin
             xyz="-0.23495 0 0.127"
@@ -303,5 +312,7 @@
         <axis
             xyz="0 0 -1" />
+        <!--
         <limit lower="-3.14" upper="3.14" effort="1500" velocity="0.5" />
+        -->
     </joint>
     <link
@@ -350,5 +361,5 @@
             link="gps_link" />
         <axis
-            xyz="0 0 0" />
+            xyz="0 0 1" />
     </joint>
     <link
@@ -360,5 +371,5 @@
             <mass
                 value="${4.0*lb}" />
-            <xacro:cylinder_inertia m="${4.0*lb}" r="${0.5*13*inch}" h="${2.5*inch}"/>
+            <xacro:cylinder_inertia m="${4.0*lb}" r="${0.5*14*inch}" h="${2.5*inch}"/>
         </inertial>
         <visual>
@@ -407,5 +418,5 @@
             <mass
                 value="${4.0*lb}" />
-            <xacro:cylinder_inertia m="${4.0*lb}" r="${0.5*13*inch}" h="${2.5*inch}"/>
+            <xacro:cylinder_inertia m="${4.0*lb}" r="${0.5*14*inch}" h="${2.5*inch}"/>
         </inertial>
         <visual>
@@ -482,5 +493,5 @@
     <joint
         name="caster_fl_joint"
-        type="continuous">
+        type="fixed">
         <origin
             xyz="0.33655 0.2667 0.0381"
@@ -529,5 +540,5 @@
     <joint
         name="caster_bl_joint"
-        type="continuous">
+        type="fixed">
         <origin
             xyz="-0.33655 0.2667 0.0381"
@@ -576,5 +587,5 @@
     <joint
         name="caster_fr_joint"
-        type="continuous">
+        type="fixed">
         <origin
             xyz="0.33655 -0.2667 0.0381"
@@ -623,5 +634,5 @@
     <joint
         name="caster_br_joint"
-        type="continuous">
+        type="fixed">
         <origin
             xyz="-0.33655 -0.2667 0.0381"
@@ -635,8 +646,18 @@
     </joint>
     <!-- transmission -->
+    <transmission name="seat_transmission">
+        <type>transmission_interface/SimpleTransmission</type>
+        <actuator name="seat_motor">
+            <hardwareInterface>hardware_interface/VelocityJointInterface</hardwareInterface>
+            <mechanicalReduction>1</mechanicalReduction>
+        </actuator>
+        <joint name="seat_joint">
+            <hardwareInterface>hardware_interface/VelocityJointInterface</hardwareInterface>
+        </joint>
+    </transmission>
     <gazebo reference="right_wheel_link">
-        <mu1 value="1.0"/>
-        <mu2 value="1.0"/>
-        <kp value="1000000.0" />
+        <mu1 value="200.0"/>
+        <mu2 value="100.0"/>
+        <kp value="10000000.0" />
         <kd value="1.0" />
         <!--<fdir1 value="1 0 0"/>-->
@@ -654,7 +675,7 @@
     </transmission>
     <gazebo reference="left_wheel_link">
-        <mu1 value="1.0"/>
-        <mu2 value="1.0"/>
-        <kp value="1000000.0" />
+        <mu1 value="200.0"/>
+        <mu2 value="100.0"/>
+        <kp value="10000000.0" />
         <kd value="1.0" />
         <!--<fdir1 value="1 0 0"/>-->
@@ -672,28 +693,28 @@
     </transmission>
     <gazebo reference="caster_fl_link">
-        <mu1 value="0.0"/>
-        <mu2 value="0.0"/>
-        <kp value="1000000.0" />
+        <mu1 value="0."/>
+        <mu2 value="0."/>
+        <kp value="100000.0" />
         <kd value="1.0" />
         <!--<fdir1 value="1 0 0"/>-->
     </gazebo>
     <gazebo reference="caster_fr_link">
-        <mu1 value="0.0"/>
-        <mu2 value="0.0"/>
-        <kp value="1000000.0" />
+        <mu1 value="0."/>
+        <mu2 value="0."/>
+        <kp value="100000.0" />
         <kd value="1.0" />
         <!--<fdir1 value="1 0 0"/>-->
     </gazebo>
     <gazebo reference="caster_bl_link">
-        <mu1 value="0.0"/>
-        <mu2 value="0.0"/>
-        <kp value="1000000.0" />
+        <mu1 value="0."/>
+        <mu2 value="0."/>
+        <kp value="100000.0" />
         <kd value="1.0" />
         <!--<fdir1 value="1 0 0"/>-->
     </gazebo>
     <gazebo reference="caster_br_link">
-        <mu1 value="0.0"/>
-        <mu2 value="0.0"/>
-        <kp value="1000000.0" />
+        <mu1 value="0."/>
+        <mu2 value="0."/>
+        <kp value="100000.0" />
         <kd value="1.0" />
         <!--<fdir1 value="1 0 0"/>-->
@@ -768,5 +789,5 @@
 				<cameraInfoTopicName>rgb/camera_info</cameraInfoTopicName>
 				<depthImageCameraInfoTopicName>depth/camera_info</depthImageCameraInfoTopicName>
-				<frameName>kinect_optical</frameName>
+				<frameName>realsense_optical</frameName>
 				<baseline>0.1</baseline>
 				<distortion_k1>0.0</distortion_k1>

Commit message: bringup and localization, start udev rules

File: pwm_description/urdf/wheelchairdev.urdf.xacro (robot description, xacro)
@@ -2,4 +2,5 @@
 <robot name="wheelchair" xmlns:xacro="http://ros.org/wiki/xacro">
 	<xacro:include filename="$(find pwm_description)/urdf/defs.urdf.xacro"/>
+    <xacro:include filename="$(find pwm_description)/urdf/wheelchairdev.gazebo"/>
     <link name="base_footprint">
     </link>
@@ -656,147 +657,3 @@
         </joint>
     </transmission>
-    <gazebo reference="right_wheel_link">
-        <mu1 value="200.0"/>
-        <mu2 value="100.0"/>
-        <kp value="10000000.0" />
-        <kd value="1.0" />
-        <!--<fdir1 value="1 0 0"/>-->
-    </gazebo>
-    <transmission name="right_wheel_transmission">
-        <type>transmission_interface/SimpleTransmission</type>
-        <!--<type>hardware_interface</type>-->
-        <actuator name="right_wheel_motor">
-            <hardwareInterface>hardware_interface/VelocityJointInterface</hardwareInterface>
-            <mechanicalReduction>1</mechanicalReduction>
-        </actuator>
-        <joint name="right_wheel_joint">
-            <hardwareInterface>hardware_interface/VelocityJointInterface</hardwareInterface>
-        </joint>
-    </transmission>
-    <gazebo reference="left_wheel_link">
-        <mu1 value="200.0"/>
-        <mu2 value="100.0"/>
-        <kp value="10000000.0" />
-        <kd value="1.0" />
-        <!--<fdir1 value="1 0 0"/>-->
-    </gazebo>
-    <transmission name="left_wheel_transmission">
-        <type>transmission_interface/SimpleTransmission</type>
-        <!--<type>hardware_interface</type>-->
-        <actuator name="left_wheel_motor">
-            <hardwareInterface>hardware_interface/VelocityJointInterface</hardwareInterface>
-            <mechanicalReduction>1</mechanicalReduction>
-        </actuator>
-        <joint name="left_wheel_joint">
-            <hardwareInterface>hardware_interface/VelocityJointInterface</hardwareInterface>
-        </joint>
-    </transmission>
-    <gazebo reference="caster_fl_link">
-        <mu1 value="0."/>
-        <mu2 value="0."/>
-        <kp value="100000.0" />
-        <kd value="1.0" />
-        <!--<fdir1 value="1 0 0"/>-->
-    </gazebo>
-    <gazebo reference="caster_fr_link">
-        <mu1 value="0."/>
-        <mu2 value="0."/>
-        <kp value="100000.0" />
-        <kd value="1.0" />
-        <!--<fdir1 value="1 0 0"/>-->
-    </gazebo>
-    <gazebo reference="caster_bl_link">
-        <mu1 value="0."/>
-        <mu2 value="0."/>
-        <kp value="100000.0" />
-        <kd value="1.0" />
-        <!--<fdir1 value="1 0 0"/>-->
-    </gazebo>
-    <gazebo reference="caster_br_link">
-        <mu1 value="0."/>
-        <mu2 value="0."/>
-        <kp value="100000.0" />
-        <kd value="1.0" />
-        <!--<fdir1 value="1 0 0"/>-->
-    </gazebo>
-	<gazebo>
-		<plugin name="gazebo_ros_control" filename="libgazebo_ros_control.so">
-			<robotNamespace>/wheelchair</robotNamespace>
-			<robotSimType>gazebo_ros_control/DefaultRobotHWSim</robotSimType>
-		</plugin>
-	</gazebo>
-    <!-- sensors -->
-	<gazebo reference="lidar_link">
-		<sensor type="ray" name="lidar">
-			<pose>0 0 0 0 0 0</pose>
-			<visualize>true</visualize> <!-- ?? -->
-			<update_rate>40</update_rate>
-			<ray>
-				<scan>
-					<horizontal>
-						<samples>1024</samples>
-						<resolution>1</resolution><!--?-->
-						<min_angle>-2.35</min_angle> <!-- +-135 deg -->
-						<max_angle>2.35</max_angle>
-					</horizontal>
-				</scan>
-				<range>
-					<min>0.06</min>
-					<max>4.0</max>
-					<resolution>0.01</resolution>
-				</range>
-				<noise>
-					<type>gaussian</type>
-					<mean>0.0</mean>
-					<stddev>0.01</stddev>
-				</noise>
-			</ray>
-			<plugin name="gazebo_ros_head_hokuyo_controller" filename="libgazebo_ros_laser.so">
-				<topicName>scan</topicName>
-				<frameName>lidar_link</frameName>
-			</plugin>
-		</sensor>
-	</gazebo>
-	<gazebo reference="realsense_link">
-		<sensor type="depth" name="kinect">
-			<always_on>true</always_on>
-			<update_rate>20.0</update_rate>
-			<camera>
-				<horizontal_fov>${60.0*deg}</horizontal_fov>
-				<image>
-					<format>B8G8R8</format>
-					<width>640</width>
-					<height>480</height>
-				</image>
-				<clip>
-					<near>0.05</near>
-					<far>8.0</far>
-				</clip>
-				<!-- WARNING : no noise in depth -->
-				<noise>
-					<type>gaussian</type>
-					<mean>0.0</mean>
-					<stddev>0.01</stddev>
-				</noise>
-			</camera>
-			<plugin name="kinect_camera_controller" filename="libgazebo_ros_openni_kinect.so">
-				<cameraName>kinect</cameraName>
-				<alwaysOn>true</alwaysOn>
-				<updateRate>10</updateRate>
-				<imageTopicName>rgb/image_raw</imageTopicName>
-				<depthImageTopicName>depth/image_raw</depthImageTopicName>
-				<pointCloudTopicName>depth/points</pointCloudTopicName>
-				<cameraInfoTopicName>rgb/camera_info</cameraInfoTopicName>
-				<depthImageCameraInfoTopicName>depth/camera_info</depthImageCameraInfoTopicName>
-				<frameName>realsense_optical</frameName>
-				<baseline>0.1</baseline>
-				<distortion_k1>0.0</distortion_k1>
-				<distortion_k2>0.0</distortion_k2>
-				<distortion_k3>0.0</distortion_k3>
-				<distortion_t1>0.0</distortion_t1>
-				<distortion_t2>0.0</distortion_t2>
-				<pointCloudCutoff>0.4</pointCloudCutoff>
-			</plugin>
-		</sensor>
-	</gazebo>
 </robot>
