Commit message: collision bbox configurations

File: pwm_description/urdf/wheelchairdev.urdf.xacro (robot description, xacro)
@@ -1,13 +1,13 @@
 <?xml version="1.0"?>
 <robot name="wheelchair" xmlns:xacro="http://ros.org/wiki/xacro">
-	<xacro:include filename="$(find pwm_description)/urdf/defs.urdf.xacro"/>
+    <xacro:include filename="$(find pwm_description)/urdf/defs.urdf.xacro"/>
     <xacro:include filename="$(find pwm_description)/urdf/wheelchairdev.gazebo"/>
     <link name="base_footprint">
     </link>
-	<joint name="base_footprint_joint" type="fixed">
-        <origin xyz="0 0 ${0.5*13*inch-0.114}" rpy="0 0 0"/>
-		<parent link="base_footprint"/>
-		<child link="base_link"/>
-	</joint>
+    <joint name="base_footprint_joint" type="fixed">
+        <origin xyz="0 0 ${0.5*14*inch-0.1143}" rpy="0 0 0"/>
+        <parent link="base_footprint"/>
+        <child link="base_link"/>
+    </joint>
     <link
         name="base_link">
@@ -35,10 +35,7 @@
         </visual>
         <collision>
-            <origin
-                xyz="0 0 0"
-                rpy="0 0 0" />
-            <geometry>
-                <mesh
-                    filename="package://pwm_description/meshes/base_link.STL" />
+            <origin xyz="0.0 0.0 0.152400001884" rpy="0 0 0"/>
+            <geometry>
+                <box size="0.711199998856 0.457199990749 0.304800003767"/>
             </geometry>
         </collision>
@@ -75,10 +72,7 @@
         </visual>
         <collision>
-            <origin
-                xyz="0 0 0"
-                rpy="0 0 0" />
-            <geometry>
-                <mesh
-                    filename="package://pwm_description/meshes/seat_link.STL" />
+            <origin xyz="-0.0635000020266 7.45058059692e-09 0.0127000026405" rpy="0 0 0"/>
+            <geometry>
+                <box size="0.660400032997 0.482599973679 0.228599995375"/>
             </geometry>
         </collision>
@@ -129,10 +123,7 @@
         </visual>
         <collision>
-            <origin
-                xyz="0 0 0"
-                rpy="0 0 0" />
-            <geometry>
-                <mesh
-                    filename="package://pwm_description/meshes/footrest_link.STL" />
+            <origin xyz="0.128881782293 -0.200304538012 0.0" rpy="0 0 0"/>
+            <geometry>
+                <box size="0.30856359005 0.400308251381 0.43180000782"/>
             </geometry>
         </collision>
@@ -185,10 +176,7 @@
         </visual>
         <collision>
-            <origin
-                xyz="0 0 0"
-                rpy="0 0 0" />
-            <geometry>
-                <mesh
-                    filename="package://pwm_description/meshes/lidar_link.STL" />
+            <origin xyz="-0.00884072016925 0.0 -0.0141306817532" rpy="0 0 0"/>
+            <geometry>
+                <box size="0.0632499977946 0.0500000007451 0.070000000298"/>
             </geometry>
         </collision>
@@ -232,10 +220,7 @@
         </visual>
         <collision>
-            <origin
-                xyz="0 0 0"
-                rpy="0 0 0" />
-            <geometry>
-                <mesh
-                    filename="package://pwm_description/meshes/realsense_link.STL" />
+            <origin xyz="-0.0125249996781 0.0 0.0" rpy="0 0 0"/>
+            <geometry>
+                <box size="0.0250499993563 0.0900000035763 0.0250000003725"/>
             </geometry>
         </collision>
@@ -256,9 +241,9 @@
     <!-- optical frame -->
     <link name="realsense_optical"/>
-	<joint name="realsense_optical_joint" type="fixed">
-		<origin xyz="0 0 0" rpy="${-pi/2} 0 ${-pi/2}"/>
-		<parent link="realsense_link"/>
-		<child link="realsense_optical"/>
-	</joint>
+    <joint name="realsense_optical_joint" type="fixed">
+        <origin xyz="0 0 0" rpy="${-pi/2} 0 ${-pi/2}"/>
+        <parent link="realsense_link"/>
+        <child link="realsense_optical"/>
+    </joint>
     <link
         name="back_link">
@@ -292,10 +277,7 @@
         </visual>
         <collision>
-            <origin
-                xyz="0 0 0"
-                rpy="0 0 0" />
-            <geometry>
-                <mesh
-                    filename="package://pwm_description/meshes/back_link.STL" />
+            <origin xyz="0.256545692682 0.355273872614 -0.0322397202253" rpy="0 0 0"/>
+            <geometry>
+                <box size="0.75830322504 0.710547745228 0.710565447807"/>
             </geometry>
         </collision>
@@ -342,10 +324,7 @@
         </visual>
         <collision>
-            <origin
-                xyz="0 0 0"
-                rpy="0 0 0" />
-            <geometry>
-                <mesh
-                    filename="package://pwm_description/meshes/gps_link.STL" />
+            <origin xyz="-0.00362478382885 0.0 0.00983087625355" rpy="0 0 0"/>
+            <geometry>
+                <box size="0.0597429461777 0.0525326915085 0.0197107437998"/>
             </geometry>
         </collision>

Commit message: finished configuring gazebo sim

File: pwm_description/urdf/wheelchairdev.urdf.xacro (robot description, xacro)
@@ -123,7 +123,17 @@
         </visual>
         <collision>
+            <!--
+                 Disabled due to lidar
             <origin xyz="0.128881782293 -0.200304538012 0.0" rpy="0 0 0"/>
             <geometry>
                 <box size="0.30856359005 0.400308251381 0.43180000782"/>
+            </geometry>
+            -->
+            <origin
+                xyz="0 0 0"
+                rpy="0 0 0" />
+            <geometry>
+                <mesh
+                    filename="package://pwm_description/meshes/footrest_link.STL" />
             </geometry>
         </collision>
@@ -371,7 +381,12 @@
                 xyz="0 0 0"
                 rpy="0 0 0" />
+            <!--
             <geometry>
                 <mesh
                     filename="package://pwm_description/meshes/right_wheel_link.STL" />
+            </geometry>
+            -->
+            <geometry>
+                <cylinder length="${2.5*inch}" radius="${0.5*14*inch}"/>
             </geometry>
         </collision>
@@ -419,6 +434,5 @@
                 rpy="0 0 0" />
             <geometry>
-                <mesh
-                    filename="package://pwm_description/meshes/left_wheel_link.STL" />
+                <cylinder length="${2.5*inch}" radius="${0.5*14*inch}"/>
             </geometry>
         </collision>
@@ -465,7 +479,12 @@
                 xyz="0 0 0"
                 rpy="0 0 0" />
+            <!--
             <geometry>
                 <mesh
                     filename="package://pwm_description/meshes/caster_fl_link.STL" />
+            </geometry>
+            -->
+            <geometry>
+                <cylinder length="${2.0*inch}" radius="${0.5*8*inch}"/>
             </geometry>
         </collision>
@@ -513,6 +532,5 @@
                 rpy="0 0 0" />
             <geometry>
-                <mesh
-                    filename="package://pwm_description/meshes/caster_bl_link.STL" />
+                <cylinder length="${2.0*inch}" radius="${0.5*8*inch}"/>
             </geometry>
         </collision>
@@ -560,6 +578,5 @@
                 rpy="0 0 0" />
             <geometry>
-                <mesh
-                    filename="package://pwm_description/meshes/caster_fr_link.STL" />
+                <cylinder length="${2.0*inch}" radius="${0.5*8*inch}"/>
             </geometry>
         </collision>
@@ -607,6 +624,5 @@
                 rpy="0 0 0" />
             <geometry>
-                <mesh
-                    filename="package://pwm_description/meshes/caster_br_link.STL" />
+                <cylinder length="${2.0*inch}" radius="${0.5*8*inch}"/>
             </geometry>
         </collision>

Commit message: working gazebo configuration (with RTABMAP)

File: pwm_description/urdf/wheelchairdev.urdf.xacro (robot description, xacro)
@@ -206,5 +206,5 @@
     </joint>
     <link
-        name="realsense_link">
+        name="camera_link">
         <inertial>
             <origin
@@ -237,5 +237,5 @@
     </link>
     <joint
-        name="realsense_joint"
+        name="camera_joint"
         type="fixed">
         <origin
@@ -245,14 +245,40 @@
             link="footrest_link" />
         <child
-            link="realsense_link" />
+            link="camera_link" />
         <axis
             xyz="0 0 1" />
     </joint>
     <!-- optical frame -->
-    <link name="realsense_optical"/>
-    <joint name="realsense_optical_joint" type="fixed">
+    <link name="camera_optical"/>
+    <joint name="camera_optical_joint" type="fixed">
         <origin xyz="0 0 0" rpy="${-pi/2} 0 ${-pi/2}"/>
-        <parent link="realsense_link"/>
-        <child link="realsense_optical"/>
+        <parent link="camera_link"/>
+        <child link="camera_optical"/>
+    </joint>
+    <!-- alignment frames -->
+    <!-- setup aliases for compatibility with realsense -->
+    <link name="camera_aligned_depth_to_color_frame"/>
+    <joint name="align_d2c" type="fixed">
+        <origin xyz="0 0 0" rpy="0 0 0"/>
+        <parent link="camera_optical"/>
+        <child link="camera_aligned_depth_to_color_frame"/>
+    </joint>
+    <link name="camera_aligned_depth_to_infra1_frame"/>
+    <joint name="align_d2i1" type="fixed">
+        <origin xyz="0 0 0" rpy="0 0 0"/>
+        <parent link="camera_optical"/>
+        <child link="camera_aligned_depth_to_infra1_frame"/>
+    </joint>
+    <link name="camera_aligned_depth_to_infra2_frame"/>
+    <joint name="align_d2i2" type="fixed">
+        <origin xyz="0 0 0" rpy="0 0 0"/>
+        <parent link="camera_optical"/>
+        <child link="camera_aligned_depth_to_infra2_frame"/>
+    </joint>
+    <link name="camera_aligned_depth_to_fisheye_frame" />
+    <joint name="align_d2f" type="fixed">
+        <origin xyz="0 0 0" rpy="0 0 0"/>
+        <parent link="camera_optical"/>
+        <child link="camera_aligned_depth_to_fisheye_frame"/>
     </joint>
     <link

Commit message: attempt at sensor fusion

File: pwm_description/urdf/wheelchairdev.urdf.xacro (robot description, xacro)
@@ -213,4 +213,30 @@
             xyz="0 0 1" />
     </joint>
+    <link name="imu">
+        <inertial>
+            <origin rpy="0 0 0" xyz="0 0 0"/>
+            <mass value="1e-2"/>
+            <xacro:box_inertia x="1e-2" y="1e-2" z="1e-2" mass="1e-2"/>
+        </inertial>
+        <visual>
+            <origin rpy="0 0 0" xyz="0 0 0"/>
+            <geometry>
+                <box size="1e-2 1e-2 1e-2"/>
+            </geometry>
+        </visual>
+        <collision>
+            <origin rpy="0 0 0" xyz="0 0 0"/>
+            <geometry>
+                <box size="1e-2 1e-2 1e-2"/>
+            </geometry>
+        </collision>
+    </link>
+    <joint name="imu_joint" type="fixed">
+        <origin xyz="0.13695 -0.32488 -0.00060405"
+            rpy="-1.5708 0 0.22" />
+        <parent link="footrest_link"/>
+        <child link="imu"/>
+        <axis xyz="1 0 0"/>
+    </joint>
     <link
         name="camera_link">
@@ -374,5 +400,5 @@
         <inertial>
             <origin
-                xyz="5.5511E-17 0 0.032142"
+                xyz="0 0 0"
                 rpy="0 0 0" />
             <mass
@@ -426,5 +452,5 @@
         <inertial>
             <origin
-                xyz="0 -2.7756E-17 -0.032142"
+                xyz="0 0 0"
                 rpy="0 0 0" />
             <mass
@@ -472,5 +498,5 @@
         <inertial>
             <origin
-                xyz="-2.2898E-16 6.9389E-18 -0.0010598"
+                xyz="0 0 0"
                 rpy="0 0 0" />
             <mass
@@ -529,5 +555,5 @@
         <inertial>
             <origin
-                xyz="1.1102E-16 -2.0817E-16 -0.0010598"
+                xyz="0 0 0"
                 rpy="0 0 0" />
             <mass
@@ -580,5 +606,5 @@
         <inertial>
             <origin
-                xyz="1.1796E-16 -2.0123E-16 0.0010598"
+                xyz="0 0 0"
                 rpy="0 0 0" />
             <mass

Commit message: phidgets imu configurations + regular imu attempts to avoid manual power-cycle

File: pwm_description/urdf/wheelchairdev.urdf.xacro (robot description, xacro)
@@ -239,4 +239,13 @@
         <axis xyz="1 0 0"/>
     </joint>
+	<!-- add phidgets -->
+	<link name="pimu">
+	</link>
+	<joint name="pimu_joint" type="fixed">
+		<origin xyz="-0.2 0.0 0.72" rpy="0 0.04 0"/>
+		<parent link="base_footprint"/>
+		<child link="pimu"/>
+		<axis xyz="1 0 0"/>
+	</joint>
     <link
         name="camera_link">
